File: Eletronics/BLE_Emergency_lights_v1.0/BLE_Emergency_lights_v1.0.brd (EAGLE design)
At the start: 100.8 x 76 mm, 168 parts, among them IC1 SI7021-, U1 LIS2DH12

Commit message: BLE_Emergency_lights_v1.0
Parts:
- added U3: VL53L0X, 0000_GV_sensors:SENSOR_VL53L0X
Connections:
- net GND: now also U3.12, U3.2, U3.3, U3.4, U3.6
- net SCL: now also U3.10
- net SDA: now also U3.9
- net SENSOR_PWR: now also U3.1, U3.11, U3.5
Routing:
- net GND: track 190.7 -> 199.2 mm, vias 8 -> 9
- net SENSOR_PWR: track 35.9 -> 44.4 mm, vias 0 -> 1
- net SDA: track 24.5 -> 31.2 mm
- net SCL: track 27.0 -> 29.8 mm, vias 2 -> 3
- net MAIN_LED_GND: track 579.4 -> 580.1 mm
